File: kicad/minitel5.sch (KiCad schematic (older format))
At the start: 441 parts, among them J1 DIN-5, J101 12V DC Input, J2 LCD Panel Connector, J201 RJ12, J202 Mini-DIN-9, J203 Speaker, J999 Keyboard Connector, Q101 IRF9Z10, Q102 BC856, Q103 NOT POPULATED, Q104 BC856, Q105 \"1B\", Q106 \"1B\", Q108 \"3B\", Q110 \"3B\", Q112 \"3B\", Q113 BD132, Q114 \"3B\", Q115 \"3B\", Q116 \"1B\", Q117 \"3B\", Q118 \"1B\", Q119 \"3B\", Q120 \"1B\", Q121 \"3B\", Q122 \"3B\", Q123 \"3B\", Q124 \"3B\", Q125 \"3B\", Q126 \"3B\", Q130 \"3B\", Q131 \"1B\", Q132 \"1B\", Q133 Q_NPN_BCE, Q134 \"1B\", Q135 \"3B\", Q136 \"1B\", Q2 \"1B\", Q201 VN2410L, Q202 \"6B\", Q203 \"6B\", Q204 \"1V\", Q205 BD232T, Q206 \"6B\", Q207 \"6B\", Q208 \"5B\", Q209 NOT POPULATED, Q211 \"1B\", Q3 \"1B\", Q4 \"1B\", Q5 \"1B\", Q6 \"3B\", Q7 \"3B\", SW101 Pushed if rechargeable Batter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, SW102 ON/OFF switch, T101 VOGT_406_47, Y1 11MHz, Y201 3.57MHz

Commit message: Updated Kicad schematics
Parts:
- added C112: 470uF 10V, symbol Device:CP
- BT1: value Battery_Cell -> 3V Backup Battery Cell
Connections:
- net MN2-53 is gone; now on net MN2-55: J999.13 (Pin_13), R20.2
- net GND: now also C112.2
- net J202_PIN1: now also C228.2
- net MN19-6: now also R162.1; no longer R162.2
- net MN2-55: no longer J999.14 (Pin_14), R19.2
- net MN2-56: now also J999.14 (Pin_14), R19.2; no longer J999.15 (Pin_15), R18.2
- net MN2-57: now also J999.15 (Pin_15), R18.2; no longer J999.16 (Pin_16), R17.2
- net MN2-58: now also J999.16 (Pin_16), R17.2; no longer J999.17 (Pin_17), R16.2
- net MN2-59: now also J999.17 (Pin_17), R16.2; no longer J999.18 (Pin_18), Q105.3 (C), R112.1
- net VEE: now also C112.1
- net ~PSEN: now also MN1.32 (~PSEN), MN3.22 (~OE)
- net VBATT_OR_8V: now reaches Q207.3 (C)
- net VBATT_OR_8V: now also C109.1, CR114.1 (K), Q104.2 (E), Q113.1 (E), R110.2, R130.2, R131.1, R138.1, RV101.2
- net ~DIN_WAKE: now reaches CR111.1 (K), CR2.1 (K), L3.2, VR2.2
- net ALIM_J1_PIN5: now reaches J1.5, Q101.2 (D), R101.2
- net MODEM_SIGNAL: now reaches C205.2, CR210.2 (A), R224.1, R226.1, TR201.1 (AA)
- net at R40.1: no longer MN2.36
- net at C221.2: now also R240.2; no longer MN2.83
- net at C107.1, C108.2, MA103.3 (CAP): now also C106.1; no longer C106.2
- net at MA103.6 (C), Q114.3 (C): now also R139.1; no longer R139.2
- net at C220.2, CR217.2 (A), CR218.1 (K)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: now also R240.1; no longer R240.2
- net BEEP: now reaches C221.1
- net BEEP: now also MN2.83; no longer R240.1
- net at CR125.1 (K), Q130.2 (E), Q132.3 (C)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: now also R163.1; no longer R163.2
- net at Q130.1 (B), R165.1: now also R163.2; no longer R163.1
- net at Q131.2 (E), R166.1, R167.1: no longer CR126.2 (A)
- net at Q134.1 (B): now also R162.2; no longer R162.1
- net at C108.1, R134.1, R136.2: now also R137.1; no longer R137.2
- net at C111.2, Q114.1 (B), R138.2: now also R139.2; no longer R139.1
- net +8V: no longer names the net of MA101.3 (VO), R160.2, RL101.10
- new net: C106.2, MA103.1 (E-), R137.2
- new net ~SPACEBAR_SW: J999.18 (Pin_18), Q105.3 (C), R112.1
- no-connect marks 32 -> 34
Other:
- note removed: "TODO"
- moved on the sheet: BT1, C10, C101, C102, C103, C104, C106, C107, C108, C109, C110, C111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
