File: kicad/minitel5.sch (KiCad schematic (older format))
At the start: 442 parts, among them J1 DIN-5, J101 12V DC Input, J2 LCD Panel Connector, J201 RJ12, J202 Mini-DIN-9, J203 Speaker, J999 Keyboard Connector, Q101 IRF9Z10, Q102 BC856, Q103 NOT POPULATED, Q104 BC856, Q105 \"1B\", Q106 \"1B\", Q108 \"3B\", Q110 \"3B\", Q112 \"3B\", Q113 BD132, Q114 \"3B\", Q115 \"3B\", Q116 \"1B\", Q117 \"3B\", Q118 \"1B\", Q119 \"3B\", Q120 \"1B\", Q121 \"3B\", Q122 \"3B\", Q123 \"3B\", Q124 \"3B\", Q125 \"3B\", Q126 \"3B\", Q130 \"3B\", Q131 \"1B\", Q132 \"1B\", Q133 Q_NPN_BCE, Q134 \"1B\", Q135 \"3B\", Q136 \"1B\", Q2 \"1B\", Q201 VN2410L, Q202 \"6B\", Q203 \"6B\", Q204 \"1V\", Q205 BD232T, Q206 \"6B\", Q207 \"6B\", Q208 \"5B\", Q209 NOT POPULATED, Q211 \"1B\", Q3 \"1B\", Q4 \"1B\", Q5 \"1B\", Q6 \"3B\", Q7 \"3B\", SW101 Pushed if rechargeable Batter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, SW102 ON/OFF switch, T101 VOGT_406_47, Y1 11MHz, Y201 3.57MHz

Commit message: Correcting some typos and smalls things in schematics
Connections:
- net NM1-5 renamed MN1-5
- net NM1-7 renamed MN1-7
- net NM1-9 renamed MN1-9
Other:
- note added: "from DECOPLAT"
- note removed: "to MN6"
Changed lines of the file:
@@
 	11950 17400 11550 17400
 Text Notes 11800 17250 2    50   ~ 0
-to MN6
+from DECOPLAT
 Wire Wire Line
 	11950 17500 11550 17500
@@
 	25850 5800 25450 5800
 Text Label 25450 5800 0    50   ~ 0
-NM1-9
+MN1-9
 Text Label 15700 16450 0    50   ~ 0
-NM1-9
+MN1-9
 $Comp
 L Device:R R150
@@
 	25850 5600 25450 5600
 Text Label 25450 5600 0    50   ~ 0
-NM1-7
+MN1-7
 Text Label 25750 8850 0    50   ~ 0
-NM1-7
+MN1-7
 Wire Wire Line
 	26650 4900 26650 4600
 Text Label 26650 4600 3    50   ~ 0
-NM1-5
+MN1-5
 Text Label 37050 15650 0    50   ~ 0
-NM1-5
+MN1-5
 Wire Wire Line
 	37050 15650 37450 15650

Commit message: Small schematic fix
Connections:
- net at CR126.2 (A): now also Q131.2 (E), R166.1, R167.1
Changed lines of the file:
@@
 $EndComp
 Wire Wire Line
-	2850 15750 4950 15750
+	2850 15750 4100 15750
 Wire Wire Line
 	2850 14300 4200 14300
@@
 Wire Wire Line
 	30500 7150 30500 9500
+Wire Wire Line
+	4100 15800 4100 15750
 Wire Bus Line
 	24850 25900 25800 25900
@@
 Wire Bus Line
 	24100 26200 24100 29100
+Connection ~ 4100 15750
+Wire Wire Line
+	4100 15750 4950 15750
 $EndSCHEMATC
